File: ESC-single-F051T8Yx.kicad_pcb (KiCad board)
At the start: 4 copper layers, 15 x 15 mm, 56 parts, among them U1 STM32F051T8Yx, U2 TPS727xxDSE, U3 SIZF360DT-T1-GE3, U4 NCP81253MNTBG, U5 SIZF360DT-T1-GE3, U6 NCP81253MNTBG, U7 SIZF360DT-T1-GE3, U8 NCP81253MNTBG

Commit message: cleanup
Parts:
- FID1, FID2: footprint 11_PSoC_FC_whoop:TestPoint_Pad_D1.0mm_dense -> footprints:TestPoint_Pad_D1.0mm_dense
- FID3, FID4, FID5, FID6, TP6, TP7, TP8: footprint 11_PSoC_FC_whoop:pad_io_1x1.5mm -> footprints:pad_io_1x1.5mm
- R10, R12, R13, R14, R15, R16, R17, R19, R20, R21, R22, R3, R4, R5, R6, R7, R8, R9: footprint ultimateFC:R_0201_0603Metric_mod -> footprints:R_0201_0603Metric_mod
- TP2, TP3: footprint 11_PSoC_FC_whoop:batt_pad_wide_relaxed -> footprints:batt_pad_wide_relaxed
- U3, U5, U7: footprint 11_PSoC_FC_whoop:PowerPair_3.3x3.3F_BWL -> footprints:PowerPair_3.3x3.3F_BWL
- U4, U6, U8: footprint 11_PSoC_FC_whoop:DFN-8-1EP_2x2mm_P0.5mm_EP0.9x1.3mm_narrow -> footprints:DFN-8-1EP_2x2mm_P0.5mm_EP0.9x1.3mm_dense
