File: ESC-single-F051T8Yx.kicad_pcb (KiCad board)
At the start: 4 copper layers, 15 x 15 mm, 56 parts, among them U1 STM32F051T8Yx, U2 TPS727xxDSE, U3 SIZF360DT-T1-GE3, U4 NCP81253MNTBG, U5 SIZF360DT-T1-GE3, U6 NCP81253MNTBG, U7 SIZF360DT-T1-GE3, U8 NCP81253MNTBG

Commit message: changed layout of gate masuring 10M resistors slightly
Parts:
- moved FID4 1.55 mm to (56.7, 64.0)
- moved R24 1.41 mm to (55.1, 63.9), turned to 90 degrees
- moved FID3 0.95 mm to (53.8, 64.0)
- moved R25 0.55 mm to (52.5, 64.0), turned to 90 degrees
Routing:
- net Net-(R19-Pad1): track 3.69 -> 2.23 mm
- net Net-(R16-Pad1): track 3.05 -> 1.97 mm
Changed lines of the file:
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@@
-(kicad_pcb (version 20171130) (host pcbnew 5.1.6-c6e7f7d~87~ubuntu18.04.1)
+(kicad_pcb (version 20171130) (host pcbnew "(5.1.4)-1")
   (general
     (thickness 1.6)
     (drawings 11)
-    (tracks 391)
+    (tracks 393)
     (zones 0)
     (modules 56)
@@
   )
   (setup
-    (last_trace_width 0.1)
+    (last_trace_width 0.125)
     (user_trace_width 0.1)
     (user_trace_width 0.125)
@@
     (solder_mask_min_width 0.05)
     (aux_axis_origin 0 0)
-    (visible_elements FFFFFF7F)
+    (visible_elements 7FFFFFFF)
     (pcbplotparams
       (layerselection 0x010fc_ffffffff)
@@
   )
   (module footprints:pad_io_1x1.5mm (layer "F.Cu_(sig)")
-    (at 58.25 64.1)
+    (at 56.7 64.05)
     (attr virtual)
     (fp_text reference FID4 (at 0 0.5) (layer F.SilkS) hide
@@
   )
   (module footprints:pad_io_1x1.5mm (layer "F.Cu_(sig)")
-    (at 54.75 64.1)
+    (at 53.8 64.05)
     (attr virtual)
     (fp_text reference FID3 (at 0 0.5) (layer F.SilkS) hide
@@
   )
   (module Resistor_SMD:R_0402_1005Metric (layer "F.Cu_(sig)")
-    (at 53 64)
+    (at 52.45 64 90)
     (descr "Resistor SMD 0402 (1005 Metric), square (rectangular) end terminal, IPC_7351 nominal, (Body size source: http://www.tortai-tech.com/upload/download/2011102023233369053.pdf), generated with kicad-footprint-generator")
     (tags resistor)
     (attr smd)
-    (fp_text reference R25 (at 0 -1.17) (layer F.SilkS) hide
-      (effects (font (size 1 1) (thickness 0.15)))
-    )
-    (fp_text value 10M (at 0 1.17) (layer F.Fab) hide
+    (fp_text reference R25 (at 0 -1.17 90) (layer F.SilkS) hide
+      (effects (font (size 1 1) (thickness 0.15)))
+    )
+    (fp_text value 10M (at 0 1.17 90) (layer F.Fab) hide
       (effects (font (size 1 1) (thickness 0.15)))
     )
@@
     (fp_line (start 0.93 -0.47) (end 0.93 0.47) (layer F.CrtYd) (width 0.05))
     (fp_line (start 0.93 0.47) (end -0.93 0.47) (layer F.CrtYd) (width 0.05))
-    (fp_text user %R (at 0 0) (layer F.Fab) hide
+    (fp_text user %R (at 0 0 90) (layer F.Fab) hide
       (effects (font (size 0.25 0.25) (thickness 0.04)))
     )
-    (pad 2 smd roundrect (at 0.485 0) (size 0.59 0.64) (layers "F.Cu_(sig)" F.Paste F.Mask) (roundrect_rratio 0.25)
+    (pad 2 smd roundrect (at 0.485 0 90) (size 0.59 0.64) (layers "F.Cu_(sig)" F.Paste F.Mask) (roundrect_rratio 0.25)
       (net 30 "Net-(R16-Pad1)"))
-    (pad 1 smd roundrect (at -0.485 0) (size 0.59 0.64) (layers "F.Cu_(sig)" F.Paste F.Mask) (roundrect_rratio 0.25)
+    (pad 1 smd roundrect (at -0.485 0 90) (size 0.59 0.64) (layers "F.Cu_(sig)" F.Paste F.Mask) (roundrect_rratio 0.25)
       (net 42 "Net-(FID5-Pad1)"))
     (model ${KISYS3DMOD}/Resistor_SMD.3dshapes/R_0402_1005Metric.wrl
@@
   )
   (module Resistor_SMD:R_0402_1005Metric (layer "F.Cu_(sig)")
-    (at 56.5 64 180)
+    (at 55.1 63.85 90)
     (descr "Resistor SMD 0402 (1005 Metric), square (rectangular) end terminal, IPC_7351 nominal, (Body size source: http://www.tortai-tech.com/upload/download/2011102023233369053.pdf), generated with kicad-footprint-generator")
     (tags resistor)
     (attr smd)
-    (fp_text reference R24 (at 0 -1.17) (layer F.SilkS) hide
-      (effects (font (size 1 1) (thickness 0.15)))
-    )
-    (fp_text value 10M (at 0 1.17) (layer F.Fab) hide
+    (fp_text reference R24 (at 0 -1.17 90) (layer F.SilkS) hide
+      (effects (font (size 1 1) (thickness 0.15)))
+    )
+    (fp_text value 10M (at 0 1.17 90) (layer F.Fab) hide
       (effects (font (size 1 1) (thickness 0.15)))
     )
@@
     (fp_line (start 0.93 -0.47) (end 0.93 0.47) (layer F.CrtYd) (width 0.05))
     (fp_line (start 0.93 0.47) (end -0.93 0.47) (layer F.CrtYd) (width 0.05))
-    (fp_text user %R (at 0 0) (layer F.Fab) hide
+    (fp_text user %R (at 0 0 90) (layer F.Fab) hide
       (effects (font (size 0.25 0.25) (thickness 0.04)))
     )
-    (pad 2 smd roundrect (at 0.485 0 180) (size 0.59 0.64) (layers "F.Cu_(sig)" F.Paste F.Mask) (roundrect_rratio 0.25)
+    (pad 2 smd roundrect (at 0.485 0 90) (size 0.59 0.64) (layers "F.Cu_(sig)" F.Paste F.Mask) (roundrect_rratio 0.25)
       (net 32 "Net-(R19-Pad1)"))
-    (pad 1 smd roundrect (at -0.485 0 180) (size 0.59 0.64) (layers "F.Cu_(sig)" F.Paste F.Mask) (roundrect_rratio 0.25)
+    (pad 1 smd roundrect (at -0.485 0 90) (size 0.59 0.64) (layers "F.Cu_(sig)" F.Paste F.Mask) (roundrect_rratio 0.25)
       (net 41 "Net-(FID4-Pad1)"))
     (model ${KISYS3DMOD}/Resistor_SMD.3dshapes/R_0402_1005Metric.wrl
@@
   (segment (start 51.9 62.5) (end 52.2 62.8) (width 0.25) (layer "B.Cu_(sig)") (net 30))
   (via (at 52.2 63) (size 0.4) (drill 0.2) (layers "F.Cu_(sig)" "B.Cu_(sig)") (net 30))
-  (segment (start 53.485 64) (end 52.885 63.4) (width 0.125) (layer "F.Cu_(sig)") (net 30))
-  (segment (start 52.6 63.4) (end 52.2 63) (width 0.125) (layer "F.Cu_(sig)") (net 30))
-  (segment (start 52.885 63.4) (end 52.6 63.4) (width 0.125) (layer "F.Cu_(sig)") (net 30))
+  (segment (start 52.45 63.25) (end 52.2 63) (width 0.125) (layer "F.Cu_(sig)") (net 30))
+  (segment (start 52.45 63.515) (end 52.45 63.25) (width 0.125) (layer "F.Cu_(sig)") (net 30))
   (segment (start 52.65 62.15) (end 52.4 61.9) (width 0.25) (layer "B.Cu_(sig)") (net 31))
   (segment (start 52.65 62.25) (end 52.65 62.15) (width 0.25) (layer "B.Cu_(sig)") (net 31))
@@
   (segment (start 54.6 63) (end 54.6 62.045) (width 0.25) (layer "F.Cu_(sig)") (net 32))
   (segment (start 54.9 62.5) (end 54.6 62.8) (width 0.25) (layer "B.Cu_(sig)") (net 32))
-  (segment (start 56.015 64) (end 56.015 63.515) (width 0.125) (layer "F.Cu_(sig)") (net 32))
-  (segment (start 55.5 63) (end 54.6 63) (width 0.125) (layer "F.Cu_(sig)") (net 32))
-  (segment (start 56.015 63.515) (end 55.5 63) (width 0.125) (layer "F.Cu_(sig)") (net 32))
+  (segment (start 54.735 63) (end 55.1 63.365) (width 0.125) (layer "F.Cu_(sig)") (net 32))
+  (segment (start 54.6 63) (end 54.735 63) (width 0.125) (layer "F.Cu_(sig)") (net 32))
   (segment (start 54.4 61.9) (end 54.9 61.9) (width 0.25) (layer "B.Cu_(sig)") (net 33))
   (segment (start 54.15 62.15) (end 54.4 61.9) (width 0.25) (layer "B.Cu_(sig)") (net 33))
@@
   (segment (start 52.08 59.32) (end 52.08 59.4) (width 0.15) (layer "B.Cu_(sig)") (net 35))
   (segment (start 53.9 63) (end 53.15 63) (width 0.125) (layer "F.Cu_(sig)") (net 35))
-  (segment (start 54.75 64) (end 54.75 63.85) (width 0.125) (layer "F.Cu_(sig)") (net 35))
-  (segment (start 54.75 63.85) (end 53.9 63) (width 0.125) (layer "F.Cu_(sig)") (net 35))
   (segment (start 52.55 58.9) (end 52.525 58.875) (width 0.15) (layer "F.Cu_(sig)") (net 35))
   (segment (start 52.92 58.9) (end 52.55 58.9) (width 0.15) (layer "F.Cu_(sig)") (net 35))
@@
   (segment (start 52.93 58.91) (end 52.92 58.9) (width 0.1) (layer "F.Cu_(sig)") (net 35))
   (segment (start 52.93 61.79) (end 52.93 58.91) (width 0.1) (layer "F.Cu_(sig)") (net 35))
+  (segment (start 54 63.1) (end 54 64.05) (width 0.125) (layer "F.Cu_(sig)") (net 35))
+  (segment (start 53.9 63) (end 54 63.1) (width 0.125) (layer "F.Cu_(sig)") (net 35))
   (segment (start 57.25 60.25) (end 57.25 59.45) (width 0.125) (layer "B.Cu_(sig)") (net 36))
   (segment (start 57.25 59.45) (end 57.6 59.45) (width 0.125) (layer "B.Cu_(sig)") (net 36))
@@
   (segment (start 57.3 55.2) (end 56.675 54.575) (width 0.125) (layer "F.Cu_(sig)") (net 40))
   (segment (start 56.675 54.575) (end 56.5 54.575) (width 0.125) (layer "F.Cu_(sig)") (net 40))
-  (segment (start 56.985 64) (end 58.25 64) (width 0.125) (layer "F.Cu_(sig)") (net 41))
-  (segment (start 51.25 64) (end 52.515 64) (width 0.125) (layer "F.Cu_(sig)") (net 42))
+  (segment (start 55.985 64.35) (end 56.335 64) (width 0.125) (layer "F.Cu_(sig)") (net 41))
+  (segment (start 55.535 64.35) (end 55.985 64.35) (width 0.125) (layer "F.Cu_(sig)") (net 41))
+  (segment (start 55.1 64.335) (end 55.52 64.335) (width 0.125) (layer "F.Cu_(sig)") (net 41))
+  (segment (start 55.52 64.335) (end 55.535 64.35) (width 0.125) (layer "F.Cu_(sig)") (net 41))
+  (segment (start 52.065 64.1) (end 51.25 64.1) (width 0.125) (layer "F.Cu_(sig)") (net 42))
+  (segment (start 52.45 64.485) (end 52.065 64.1) (width 0.125) (layer "F.Cu_(sig)") (net 42))
   (zone (net 3) (net_name GND) (layer "In2.Cu_(Gnd)") (hatch edge 0.508)
     (connect_pads yes (clearance 0.15))

Commit message: update schematic, pdf, layout add 3d view PNGs
Parts:
- added C13: CP_Small, Capacitor_Tantalum_SMD:CP_EIA-3216-18_Kemet-A, F.Cu at (54.8, 51.5)
- added C14: CP_Small, Capacitor_Tantalum_SMD:CP_EIA-3216-18_Kemet-A, F.Cu at (53.8, 53.8)
- moved FID5 12.9 mm to (64.1, 63.8), turned to 90 degrees
- moved TP2 12.0 mm to (61.5, 65.0), turned to 0 degrees
- moved R25 11.6 mm to (64.0, 62.5), turned to 180 degrees
- moved FID6 11.1 mm to (64.1, 53.2), turned to 90 degrees
- moved TP3 10.8 mm to (56.0, 65.0), turned to 0 degrees
- moved FID3 10.6 mm to (64.0, 61.2), turned to 90 degrees
- moved R16 10.3 mm to (62.2, 63.1), turned to 180 degrees
- moved R6 10.3 mm to (62.2, 51.9), turned to 180 degrees
- moved R24 9.60 mm to (63.9, 59.9), turned to 180 degrees
- moved TP6 9.43 mm to (51.0, 59.0), turned to 90 degrees
- moved TP8 9.43 mm to (51.0, 56.0), turned to 90 degrees
- moved FID4 9.33 mm to (64.0, 58.3), turned to 90 degrees
- moved TP7 9.19 mm to (51.0, 57.5), turned to 90 degrees
- moved FID2 8.75 mm to (53.0, 61.8), turned to 180 degrees
- moved C6 8.57 mm to (59.7, 51.9), turned to 180 degrees
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Routing:
- net GND: track 33.7 -> 36.0 mm, vias 16 -> 18
- net 3V3_route: track 7.39 -> 8.65 mm
- net +5V: track 12.0 -> 13.1 mm, vias 6 -> 7
