File: ESC-single-F051T8Yx.sch (KiCad schematic (older format))
At the start: 56 parts, among them U1 STM32F051T8Yx, U2 TPS727xxDSE, U3 SIZF360DT-T1-GE3, U4 NCP81253MNTBG, U5 SIZF360DT-T1-GE3, U6 NCP81253MNTBG, U7 SIZF360DT-T1-GE3, U8 NCP81253MNTBG

Commit message: cleanup
Parts:
- FID1, FID2: footprint 11_PSoC_FC_whoop:TestPoint_Pad_D1.0mm_dense -> footprints:TestPoint_Pad_D1.0mm_dense
- FID3, FID4, FID5, FID6, TP6, TP7, TP8: footprint 11_PSoC_FC_whoop:pad_io_1x1.5mm -> footprints:pad_io_1x1.5mm
- R10, R12, R13, R14, R15, R16, R17, R19, R20, R21, R22, R3, R4, R5, R6, R7, R8, R9: footprint ultimateFC:R_0201_0603Metric_mod -> footprints:R_0201_0603Metric_mod
- TP2, TP3: footprint 11_PSoC_FC_whoop:batt_pad_wide_relaxed -> footprints:batt_pad_wide_relaxed
- U2: symbol lib_ultimateFC:TPS727xxDSE -> symbols:TPS727xxDSE
- U3, U5, U7: footprint 11_PSoC_FC_whoop:PowerPair_3.3x3.3F_BWL -> footprints:PowerPair_3.3x3.3F_BWL; symbol lib_ultimateFC:SIZF360DT-T1-GE3 -> symbols:SIZF360DT-T1-GE3
- U4, U6, U8: footprint 11_PSoC_FC_whoop:DFN-8-1EP_2x2mm_P0.5mm_EP0.9x1.3mm_narrow -> footprints:DFN-8-1EP_2x2mm_P0.5mm_EP0.9x1.3mm_dense; symbol lib_ultimateFC:NCP81253MNTBG -> symbols:NCP81253MNTBG

Commit message: update schematic, pdf, layout add 3d view PNGs
Parts:
- added C13, C14: CP_Small, Capacitor_Tantalum_SMD:CP_EIA-3216-18_Kemet-A, symbol Device:CP_Small
Connections:
- net +3V3: now also C14.1
- net +5V: now also C13.1
- net GND: now also C13.2, C14.2
- no-connect marks 0 -> 2
Other:
- moved on the sheet: C12
Changed lines of the file:
@@
 Sheet 1 1
 Title "halariESC"
-Date "2021-04-08"
+Date "2021-04-10"
 Rev "v0.1"
 Comp "crteensy"
@@
 L power:+5V #PWR0124
 U 1 1 607C5C6D
-P 3300 1050
-F 0 "#PWR0124" H 3300 900 50  0001 C CNN
-F 1 "+5V" H 3315 1223 50  0000 C CNN
-F 2 "" H 3300 1050 50  0001 C CNN
-F 3 "" H 3300 1050 50  0001 C CNN
-	1    3300 1050
+P 2950 1050
+F 0 "#PWR0124" H 2950 900 50  0001 C CNN
+F 1 "+5V" H 2965 1223 50  0000 C CNN
+F 2 "" H 2950 1050 50  0001 C CNN
+F 3 "" H 2950 1050 50  0001 C CNN
+	1    2950 1050
 	1    0    0    -1
 $EndComp
@@
 L power:+3V3 #PWR0125
 U 1 1 607C7982
-P 4600 1050
-F 0 "#PWR0125" H 4600 900 50  0001 C CNN
-F 1 "+3V3" H 4615 1223 50  0000 C CNN
-F 2 "" H 4600 1050 50  0001 C CNN
-F 3 "" H 4600 1050 50  0001 C CNN
-	1    4600 1050
-	1    0    0    -1
-$EndComp
-Wire Wire Line
-	4600 1050 4600 1150
+P 4950 1050
+F 0 "#PWR0125" H 4950 900 50  0001 C CNN
+F 1 "+3V3" H 4965 1223 50  0000 C CNN
+F 2 "" H 4950 1050 50  0001 C CNN
+F 3 "" H 4950 1050 50  0001 C CNN
+	1    4950 1050
+	1    0    0    -1
+$EndComp
+Wire Wire Line
+	4950 1050 4950 1150
 Wire Wire Line
 	4600 1150 4500 1150
@@
 Wire Wire Line
 	4600 1150 4600 1250
-Connection ~ 4600 1150
 $Comp
 L power:GND #PWR0146
@@
 $EndComp
 Wire Wire Line
-	4600 1750 4600 1450
+	4600 1750 4600 1550
 $Comp
 L symbols:SIZF360DT-T1-GE3 U3
@@
 Wire Wire Line
 	8050 5300 8050 5400
-$Comp
-L Device:C_Small C12
-U 1 1 615A2B93
-P 3300 1300
-F 0 "C12" H 3392 1346 50  0000 L CNN
-F 1 "1u" H 3392 1255 50  0000 L CNN
-F 2 "Capacitor_SMD:C_0402_1005Metric" H 3300 1300 50  0001 C CNN
-F 3 "~" H 3300 1300 50  0001 C CNN
-	1    3300 1300
-	1    0    0    -1
-$EndComp
 Wire Wire Line
 	3600 1450 3600 1150
-Wire Wire Line
-	3300 1400 3300 1750
 $Comp
 L power:GND #PWR0147
@@
 $EndComp
 Wire Wire Line
-	3300 1050 3300 1150
-Wire Wire Line
 	3300 1150 3600 1150
-Connection ~ 3300 1150
-Wire Wire Line
-	3300 1150 3300 1200
+Wire Wire Line
+	3300 1150 3300 1250
 Connection ~ 3600 1150
 Wire Wire Line
@@
 	9250 5900 9250 6000
 Connection ~ 9050 5900
+$Comp
+L Device:CP_Small C13
+U 1 1 608BC6D0
+P 2950 1350
+F 0 "C13" H 3038 1396 50  0000 L CNN
+F 1 "CP_Small" H 3038 1305 50  0000 L CNN
+F 2 "Capacitor_Tantalum_SMD:CP_EIA-3216-18_Kemet-A" H 2950 1350 50  0001 C CNN
+F 3 "~" H 2950 1350 50  0001 C CNN
+	1    2950 1350
+	1    0    0    -1
+$EndComp
+Wire Wire Line
+	2950 1050 2950 1150
+Wire Wire Line
+	2950 1150 3300 1150
+Connection ~ 2950 1150
+Wire Wire Line
+	2950 1150 2950 1250
+Connection ~ 3300 1150
+Wire Wire Line
+	3300 1450 3300 1550
+$Comp
+L Device:C_Small C12
+U 1 1 615A2B93
+P 3300 1350
+F 0 "C12" H 3392 1396 50  0000 L CNN
+F 1 "1u" H 3392 1305 50  0000 L CNN
+F 2 "Capacitor_SMD:C_0402_1005Metric" H 3300 1350 50  0001 C CNN
+F 3 "~" H 3300 1350 50  0001 C CNN
+	1    3300 1350
+	1    0    0    -1
+$EndComp
+Wire Wire Line
+	2950 1450 2950 1550
+Wire Wire Line
+	2950 1550 3300 1550
+Connection ~ 3300 1550
+Wire Wire Line
+	3300 1550 3300 1750
+NoConn ~ 4400 4900
+NoConn ~ 3300 4800
+$Comp
+L Device:CP_Small C14
+U 1 1 6093E24A
+P 4950 1350
+F 0 "C14" H 5038 1396 50  0000 L CNN
+F 1 "CP_Small" H 5038 1305 50  0000 L CNN
+F 2 "Capacitor_Tantalum_SMD:CP_EIA-3216-18_Kemet-A" H 4950 1350 50  0001 C CNN
+F 3 "~" H 4950 1350 50  0001 C CNN
+	1    4950 1350
+	1    0    0    -1
+$EndComp
+Wire Wire Line
+	4600 1150 4950 1150
+Connection ~ 4600 1150
+Wire Wire Line
+	4950 1150 4950 1250
+Connection ~ 4950 1150
+Wire Wire Line
+	4600 1550 4950 1550
+Wire Wire Line
+	4950 1550 4950 1450
+Connection ~ 4600 1550
+Wire Wire Line
+	4600 1550 4600 1450
 $EndSCHEMATC

Commit message: overall update
Parts:
- C13, C14: footprint Capacitor_Tantalum_SMD:CP_EIA-3216-18_Kemet-A -> Capacitor_Tantalum_SMD:CP_EIA-3528-12_Kemet-T
- TP2, TP3: footprint footprints:batt_pad_wide_relaxed -> TestPoint:TestPoint_Pad_2.5x2.5mm
- U3, U5, U7: footprint footprints:PowerPair_3.3x3.3F_BWL -> footprints:PowerPair_3.3x3.3F_BWL_mod
Changed lines of the file:
@@
 Sheet 1 1
 Title "halariESC"
-Date "2021-04-10"
+Date "2021-04-11"
 Rev "v0.1"
 Comp "crteensy"
@@
 F 0 "TP3" H 1010 1294 50  0000 L CNN
 F 1 "TestPoint_Flag" H 1010 1203 50  0000 L CNN
-F 2 "footprints:batt_pad_wide_relaxed" H 950 1200 50  0001 C CNN
+F 2 "TestPoint:TestPoint_Pad_2.5x2.5mm" H 950 1200 50  0001 C CNN
 F 3 "~" H 950 1200 50  0001 C CNN
 	1    750  1200
@@
 F 0 "TP2" H 1150 850 50  0000 R CNN
 F 1 "TestPoint_Flag" H 1550 950 50  0000 R CNN
-F 2 "footprints:batt_pad_wide_relaxed" H 950 850 50  0001 C CNN
+F 2 "TestPoint:TestPoint_Pad_2.5x2.5mm" H 950 850 50  0001 C CNN
 F 3 "~" H 950 850 50  0001 C CNN
 	1    750  850
@@
 F 0 "U3" H 9150 1750 50  0000 L CNN
 F 1 "SIZF360DT-T1-GE3" H 9200 1650 50  0000 L CNN
-F 2 "footprints:PowerPair_3.3x3.3F_BWL" H 9650 1800 50  0001 C CNN
+F 2 "footprints:PowerPair_3.3x3.3F_BWL_mod" H 9650 1800 50  0001 C CNN
 F 3 "" H 9650 1800 50  0001 C CNN
 	1    9050 1500
@@
 F 0 "U5" H 9150 3650 50  0000 L CNN
 F 1 "SIZF360DT-T1-GE3" H 9200 3550 50  0000 L CNN
-F 2 "footprints:PowerPair_3.3x3.3F_BWL" H 9650 3700 50  0001 C CNN
+F 2 "footprints:PowerPair_3.3x3.3F_BWL_mod" H 9650 3700 50  0001 C CNN
 F 3 "" H 9650 3700 50  0001 C CNN
 	1    9050 3400
@@
 F 0 "U7" H 9150 5550 50  0000 L CNN
 F 1 "SIZF360DT-T1-GE3" H 9200 5450 50  0000 L CNN
-F 2 "footprints:PowerPair_3.3x3.3F_BWL" H 9650 5600 50  0001 C CNN
+F 2 "footprints:PowerPair_3.3x3.3F_BWL_mod" H 9650 5600 50  0001 C CNN
 F 3 "" H 9650 5600 50  0001 C CNN
 	1    9050 5300
@@
 F 0 "C13" H 3038 1396 50  0000 L CNN
 F 1 "CP_Small" H 3038 1305 50  0000 L CNN
-F 2 "Capacitor_Tantalum_SMD:CP_EIA-3216-18_Kemet-A" H 2950 1350 50  0001 C CNN
+F 2 "Capacitor_Tantalum_SMD:CP_EIA-3528-12_Kemet-T" H 2950 1350 50  0001 C CNN
 F 3 "~" H 2950 1350 50  0001 C CNN
 	1    2950 1350
@@
 F 0 "C14" H 5038 1396 50  0000 L CNN
 F 1 "CP_Small" H 5038 1305 50  0000 L CNN
-F 2 "Capacitor_Tantalum_SMD:CP_EIA-3216-18_Kemet-A" H 4950 1350 50  0001 C CNN
+F 2 "Capacitor_Tantalum_SMD:CP_EIA-3528-12_Kemet-T" H 4950 1350 50  0001 C CNN
 F 3 "~" H 4950 1350 50  0001 C CNN
 	1    4950 1350
